Commit message: putting everything into packages

File: picksie_simulation/resources/robots/youbot.urdf.xacro (robot description, xacro)
@@ -21,6 +21,6 @@
   <xacro:include filename="$(find youbot_description)/urdf/materials.urdf.xacro" />
   <!-- sensors -->
-  <xacro:include filename="$(find youbot_description)/urdf/sensors/hokuyo_urg04_laser.urdf.xacro"/>
-<xacro:include filename="$(find youbot_description)/urdf/sensors/microsoft_lifecam.urdf.xacro"/>
+  <xacro:include filename="$(find picksie_simulation)/resources/urdf/sensors/hokuyo_urg04_laser.urdf.xacro"/>
+  <xacro:include filename="$(find picksie_simulation)/resources/urdf/sensors/microsoft_lifecam.urdf.xacro"/>
   <!-- Now we can start using the macros xacro:included above to define the actual youbot -->
   <!-- The first use of a macro.  This one was defined in base.urdf.xacro above.
@@ -43,10 +43,11 @@
   </xacro:youbot_gripper>
   <!-- base laser front -->
- <!-- <xacro:hokuyo_urg04_laser name="base_laser_front" parent="base" ros_topic="base_scan" update_rate="10" min_angle="-1.57" max_angle="1.57">
+  <xacro:hokuyo_urg04_laser name="base_laser_front" parent="base" ros_topic="base_scan" update_rate="10" min_angle="-1.57" max_angle="1.57">
     <origin xyz="0.3 0 -0.03" rpy="0 0 0"/>
-  </xacro:hokuyo_urg04_laser> -->
+  </xacro:hokuyo_urg04_laser>
 <!-- microsoft lifecam -->
   <xacro:microsoft_lifecam name="lifecam" parent="arm_link_5">
-    <origin xyz="0.5 0 -0.03" rpy="0 0 0"/>
+    <!--<origin xyz="0.0 0 -0.03" rpy="0 1.5707963268 0"/>-->
+    <origin xyz="-0.09 0.0 -0.02" rpy="0 -1.5707963268 0"/>
   </xacro:microsoft_lifecam>
 </robot>

Commit message: origin

File: picksie_simulation/resources/robots/youbot.urdf.xacro (robot description, xacro)
@@ -48,6 +48,5 @@
 <!-- microsoft lifecam -->
   <xacro:microsoft_lifecam name="lifecam" parent="arm_link_5">
-    <!--<origin xyz="0.0 0 -0.03" rpy="0 1.5707963268 0"/>-->
-    <origin xyz="-0.09 0.0 -0.02" rpy="0 -1.5707963268 0"/>
+    <origin xyz="-0.088 0.0 -0.02" rpy="0 -2.97 0"/>
   </xacro:microsoft_lifecam>
 </robot>

Commit message: Fixed camera model

File: picksie_simulation/resources/robots/youbot.urdf.xacro (robot description, xacro)
@@ -48,5 +48,5 @@
 <!-- microsoft lifecam -->
   <xacro:microsoft_lifecam name="lifecam" parent="arm_link_5">
-    <origin xyz="-0.088 0.0 -0.02" rpy="0 -2.97 0"/>
+    <origin xyz="-0.077 0.0 0.03" rpy="0 -1.56 0"/>
   </xacro:microsoft_lifecam>
 </robot>

File: picksie_simulation/resources/urdf/sensors/microsoft_lifecam.urdf.xacro (robot description, xacro)
@@ -23,13 +23,13 @@
       <origin xyz="-0.04 -0.0035 -0.031" rpy="${M_PI/2} 0 ${M_PI/2}" />
       <geometry>
-       <mesh filename="package://youbot_description/meshes/sensors/microsoft_lifecam.dae" scale="0.001 0.001 0.001"/>
+       <mesh filename="package://picksie_simulation/resources/meshes/sensors/microsoft_lifecam_02.dae" scale="0.001 0.001 0.001"/>
       </geometry>
     </visual>
-    <collision>
+    <!--<collision>
       <origin xyz="-0.04 -0.0035 -0.031" rpy="${M_PI/2} 0 ${M_PI/2}" />
       <geometry>
         <mesh filename="package://youbot_description/meshes/sensors/microsoft_lifecam.dae" scale="0.001 0.001 0.001"/>
       </geometry>
-    </collision>
+    </collision>-->
   </link>
   <!-- for simulation -->
