Commit message: removed backup files

File: picksie_simulation/resources/worlds/urdf/youbot_world_02.urdf (robot description, URDF)
Before this commit: robot youbot_world_02, 1 links, 0 joints
Links:
- added link base, mass 1.0; collision box size=0.1 0.1 0.02; visual box size=0.1 0.1 0.02
- added link stick, mass 1.0; collision box size=0.01 0.01 0.4; visual box size=0.01 0.01 0.4
- link box1: geometry collision mesh filename=package://picksie_simulation/resources/meshes/custom/cube02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; visual mesh filename=package://picksie_simulation/resources/meshes/custom/cube02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
Joints:
- added joint join1: type fixed, parent stick, child box1, origin xyz=0 0 0.2 rpy=0 0 0
- added joint join2: type fixed, parent stick, child base, origin xyz=0 0 -0.2 rpy=0 0 0
